File: hw/RP2040_minimal.kicad_sch (KiCad schematic)
At the start: 61 parts, among them J1 USB_C_Receptacle_USB2.0, J2 Conn_01x02, SW1 LEFT_G, SW10 RIGHT_G, SW11 RIGHT_START, SW12 MACRO_1, SW2 LEFT_START, SW3 RIGHT_R, SW4 RIGHT_B, SW5 RIGHT_WALL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

Commit message: hw: Add linear potentiometer
Parts:
- RV1: value Slider -> PTA4543-2015DPB103; footprint (none) -> PTAXX33:PTAXX43
Connections:
- net GND: now also D10.2 (VSS)
- net LED_DIN: now reaches D1.3 (DIN)
Changed lines of the file:
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@@
   (junction (at 290.83 119.38) (diameter 0) (color 0 0 0 0)
+  )
+  (junction (at 375.92 243.84) (diameter 0) (color 0 0 0 0)
   )
   (junction (at 269.24 72.39) (diameter 0) (color 0 0 0 0)
@@
     (stroke (width 0) (type default) (color 0 0 0 0))
   )
-  (wire (pts (xy 78.74 138.43) (xy 78.74 139.7))
+  (wire (pts (xy 78.74 138.43) (xy 78.74 142.24))
     (stroke (width 0) (type default) (color 0 0 0 0))
   )
@@
     (stroke (width 0) (type default) (color 0 0 0 0))
   )
+  (wire (pts (xy 375.92 243.84) (xy 393.7 243.84))
+    (stroke (width 0) (type default) (color 0 0 0 0))
+  )
   (wire (pts (xy 74.93 30.48) (xy 85.09 30.48))
     (stroke (width 0) (type default) (color 0 0 0 0))
@@
     (stroke (width 0) (type default) (color 0 0 0 0))
   )
+  (wire (pts (xy 393.7 241.3) (xy 393.7 243.84))
+    (stroke (width 0) (type default) (color 0 0 0 0))
+  )
   (wire (pts (xy 44.45 218.44) (xy 44.45 228.6))
     (stroke (width 0) (type default) (color 0 0 0 0))
@@
   )
   (wire (pts (xy 207.01 81.28) (xy 210.82 81.28))
+    (stroke (width 0) (type default) (color 0 0 0 0))
+  )
+  (wire (pts (xy 213.36 233.68) (xy 226.06 233.68))
     (stroke (width 0) (type default) (color 0 0 0 0))
   )
@@
   (label "GPIO26_ADC0" (at 245.11 180.34 180)
     (effects (font (size 1.27 1.27)) (justify right bottom))
+  )
+  (label "LED_DIN" (at 213.36 233.68 0)
+    (effects (font (size 1.27 1.27)) (justify left bottom))
   )
   (label "RUN" (at 152.4 165.1 0)
@@
     (pin "1")
   )
-  (symbol (lib_id "power:GND") (at 78.74 139.7 0) (unit 1)
-    (in_bom yes) (on_board yes)
-    (property "Reference" "#PWR08" (id 0) (at 78.74 146.05 0)
-      (effects (font (size 1.27 1.27)) hide)
-    )
-    (property "Value" "GND" (id 1) (at 74.93 140.97 0))
-    (property "Footprint" "" (id 2) (at 78.74 139.7 0)
-      (effects (font (size 1.27 1.27)) hide)
-    )
-    (property "Datasheet" "" (id 3) (at 78.74 139.7 0)
+  (symbol (lib_id "power:GND") (at 78.74 142.24 0) (unit 1)
+    (in_bom yes) (on_board yes)
+    (property "Reference" "#PWR08" (id 0) (at 78.74 148.59 0)
+      (effects (font (size 1.27 1.27)) hide)
+    )
+    (property "Value" "GND" (id 1) (at 74.93 143.51 0))
+    (property "Footprint" "" (id 2) (at 78.74 142.24 0)
+      (effects (font (size 1.27 1.27)) hide)
+    )
+    (property "Datasheet" "" (id 3) (at 78.74 142.24 0)
       (effects (font (size 1.27 1.27)) hide)
     )
@@
       (effects (font (size 1.27 1.27)) (justify right))
     )
-    (property "Value" "Slider" (id 1) (at 261.62 181.6099 0)
+    (property "Value" "PTA4543-2015DPB103" (id 1) (at 261.62 181.6099 0)
       (effects (font (size 1.27 1.27)) (justify right))
     )
-    (property "Footprint" "" (id 2) (at 259.08 180.34 0)
+    (property "Footprint" "PTAXX33:PTAXX43" (id 2) (at 259.08 180.34 0)
       (effects (font (size 1.27 1.27)) hide)
     )
@@
     )
     (path "/9644aeb8-cb0f-426e-9feb-5b87bc36a2eb"
-      (reference "RV1") (unit 1) (value "Slider") (footprint "")
+      (reference "RV1") (unit 1) (value "PTA4543-2015DPB103") (footprint "PTAXX33:PTAXX43")
     )
     (path "/85b27939-eeef-4f7b-80cd-85baaa5a0257"
