File: hw/minigeki.kicad_pcb (KiCad board)
At the start: 2 copper layers, 151.8 x 78.3 mm, 64 parts, among them J1 USB_C_Receptacle_USB2.0, J2 Conn_01x02, SW1 LEFT_R, SW10 RIGHT_WALL, SW11 MACRO_1, SW12 MACRO_2, SW2 LEFT_G, SW3 LEFT_B, SW4 LEFT_START, SW5 LEFT_WALL, SW6 RIGHT_R, SW7 RIGHT_G, SW8 RIGHT_B, SW9 RIGHT_START, U1 NCP1117-3.3_SOT223, U2 W25Q128JVS, U3 RP2040, Y1 ABLS-12.000MHZ-B4-T

Commit message: hw: add mounting holes, flip components to top of the board
Parts:
- added H1: MountingHole_Pad, MountingHole:MountingHole_2.2mm_M2_Pad_TopOnly, F.Cu at (31.0, 70.1)
- added H2: MountingHole_Pad, MountingHole:MountingHole_2.2mm_M2_Pad_TopOnly, F.Cu at (172.7, 70.1)
- added H3: MountingHole_Pad, MountingHole:MountingHole_2.2mm_M2_Pad_TopOnly, F.Cu at (172.7, 138.7)
- added H4: MountingHole_Pad, MountingHole:MountingHole_2.2mm_M2_Pad_TopOnly, F.Cu at (31.0, 138.2)
- added H5: MountingHole_Pad, MountingHole:MountingHole_2.2mm_M2_Pad_TopOnly, F.Cu at (84.3, 91.9)
- added H6: MountingHole_Pad, MountingHole:MountingHole_2.2mm_M2_Pad_TopOnly, F.Cu at (119.9, 91.9)
- C1, C10, C11, C12, C13, C14, C15, C16, C18, C2, C25, C3, C4, C5, C6, C7, C8, C9, D2, D9, J1, J2, R1, R2, R3, R4, R5, R6, R7, U1, U2, U3, Y1: moved to F.Cu
- moved C4 18.8 mm to (109.7, 89.1), turned to 0 degrees
- moved R2 18.6 mm to (91.9, 82.4)
- moved U1 16.7 mm to (108.7, 82.9)
- moved C1 16.6 mm to (108.6, 76.6), turned to 0 degrees
- moved R1 15.5 mm to (93.5, 82.4)
- moved R6 14.5 mm to (107.6, 70.4)
- moved C12 13.7 mm to (107.2, 101.3), turned to 0 degrees
- moved C15 13.7 mm to (107.2, 96.1), turned to 0 degrees
- moved C16 13.7 mm to (107.2, 94.7), turned to 0 degrees
- moved U2 13.2 mm to (93.8, 87.4), turned to 0 degrees
- moved J2 12.5 mm to (94.1, 77.4)
- moved C11 12.3 mm to (94.2, 97.1), turned to 180 degrees
- moved C13 12.3 mm to (94.2, 101.3), turned to 180 degrees
- moved R7 10.4 mm to (95.1, 70.4)
- moved C10 8.70 mm to (104.7, 93.6)
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Routing:
- net /MACRO2: track 54.5 -> 8.38 mm, vias 1 -> 0
- net /RIGHT_START: track 32.6 -> 0.00 mm
- net /LEFT_START: track 35.2 -> 4.91 mm
- net /RIGHT_R: track 29.9 -> 0.00 mm
- net /LEFT_B: track 33.4 -> 3.71 mm
- net /RIGHT_WALL: track 50.3 -> 22.2 mm
- net /LEFT_R: track 74.1 -> 46.1 mm
- net /RIGHT_G: track 41.0 -> 14.3 mm
- net /MACRO_1: track 52.0 -> 25.4 mm, vias 1 -> 0
- net /LEFT_G: track 51.5 -> 25.3 mm
- net /RIGHT_B: track 60.0 -> 34.2 mm
- net /LED_DIN: track 49.6 -> 24.6 mm, vias 1 -> 0
- net +3V3: track 64.1 -> 41.0 mm
- net Net-(D2-Pad1): track 30.8 -> 7.77 mm, vias 1 -> 0
- net Net-(D8-Pad1): track 33.4 -> 11.9 mm, vias 1 -> 0
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- added copper zone on F.Cu, net +1V1
- added copper zone on F.Cu, net +3V3
- added copper zone on F.Cu, net VBUS
- removed copper zone on B.Cu, net +1V1
- removed copper zone on B.Cu, net +3V3
- removed copper zone on B.Cu, net VBUS
Other:
- outline, holes or cut-outs redrawn

Commit message: hw: final PCB for v3.0
Parts:
- moved C10 50.1 mm to (152.3, 78.1)
- moved C6 50.1 mm to (147.3, 77.1)
- moved C7 50.1 mm to (149.8, 91.1)
- moved C8 50.1 mm to (151.3, 78.1)
- moved C9 50.1 mm to (148.3, 77.1)
- moved D5 50.1 mm to (130.2, 119.1)
- moved J2 50.1 mm to (141.7, 61.9)
- moved R1 50.1 mm to (141.1, 66.9)
- moved R2 50.1 mm to (139.6, 66.9)
- moved R3 50.1 mm to (149.3, 78.1)
- moved R4 50.1 mm to (150.3, 78.1)
- moved U1 50.1 mm to (156.3, 67.4)
- moved U3 50.1 mm to (148.3, 84.6)
- moved C1 50.1 mm to (156.3, 61.1)
- moved C22 50.1 mm to (167.6, 122.3)
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Connections:
- U3 pad 15: /RIGHT_B -> unconnected-(U3-Pad15)
- U3 pad 16: /RIGHT_G -> unconnected-(U3-Pad16)
- U3 pad 17: /RIGHT_R -> unconnected-(U3-Pad17)
- U3 pad 2: unconnected-(U3-Pad2) -> /LEFT_START
- U3 pad 29: /LEFT_B -> /RIGHT_R
- U3 pad 3: unconnected-(U3-Pad3) -> /LED_DIN
- U3 pad 30: /LEFT_G -> /RIGHT_G
- U3 pad 31: /LEFT_R -> /RIGHT_B
- U3 pad 32: unconnected-(U3-Pad32) -> /MACRO2
- U3 pad 34: unconnected-(U3-Pad34) -> /RIGHT_WALL
- U3 pad 35: unconnected-(U3-Pad35) -> /RIGHT_START
- U3 pad 36: /LED_DIN -> unconnected-(U3-Pad36)
- U3 pad 39: /MACRO_1 -> unconnected-(U3-Pad39)
- U3 pad 4: unconnected-(U3-Pad4) -> /LEFT_WALL
- U3 pad 40: /LEFT_WALL -> unconnected-(U3-Pad40)
- U3 pad 41: /LEFT_START -> unconnected-(U3-Pad41)
- U3 pad 5: unconnected-(U3-Pad5) -> /MACRO_1
- U3 pad 6: /RIGHT_START -> /LEFT_R
- U3 pad 7: /RIGHT_WALL -> /LEFT_G
- U3 pad 8: /MACRO2 -> /LEFT_B
Routing:
- net /MACRO2: track 8.38 -> 53.3 mm
- net /LEFT_B: track 3.71 -> 42.0 mm, vias 0 -> 1
- net /GPIO26_ADC0: track 7.18 -> 42.5 mm, vias 0 -> 1
- net /LEFT_START: track 4.91 -> 39.9 mm, vias 0 -> 1
- net /RIGHT_START: track 0.00 -> 34.5 mm, vias 0 -> 1
- net +3V3: track 41.0 -> 72.0 mm, vias 2 -> 6
- net /RIGHT_WALL: track 22.2 -> 52.1 mm, vias 0 -> 1
- net GND: track 115.6 -> 85.9 mm, vias 60 -> 61
- net /LEFT_G: track 25.3 -> 54.3 mm, vias 0 -> 1
- net /RIGHT_R: track 0.00 -> 28.5 mm, vias 0 -> 1
- net /MACRO_1: track 25.4 -> 52.5 mm
- net /LEFT_R: track 46.1 -> 73.0 mm, vias 0 -> 1
- net /RIGHT_B: track 34.2 -> 59.5 mm, vias 0 -> 1
- net /RIGHT_G: track 14.3 -> 39.3 mm, vias 0 -> 1
- net /LED_DIN: track 24.6 -> 49.0 mm
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Other:
- outline, holes or cut-outs redrawn
- board text removed: "GND"
