File: hw/minigeki.kicad_pcb (KiCad board)
At the start: 2 copper layers, 151.8 x 78.3 mm, 70 parts, among them J1 USB_C_Receptacle_USB2.0, J2 Conn_01x02, SW1 LEFT_R, SW10 RIGHT_WALL, SW11 MACRO_1, SW12 MACRO_2, SW2 LEFT_G, SW3 LEFT_B, SW4 LEFT_START, SW5 LEFT_WALL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

Commit message: hw: final prototype export
Parts:
- removed SW11: MACRO_1, Button_Switch_SMD:SW_SPST_PTS810
- removed SW12: MACRO_2, Button_Switch_SMD:SW_SPST_PTS810
- Y1: value ABLS-12.000MHZ-B4-T -> Q22FA23V0041800; footprint RP2040_minimal:Crystal_SMD_HC49-US -> Crystal:Crystal_SMD_3225-4Pin_3.2x2.5mm
- moved Y1 0.72 mm to (146.2, 97.0)
Connections:
- U3 pad 32: /MACRO2 -> unconnected-(U3-Pad32)
- U3 pad 5: /MACRO_1 -> unconnected-(U3-Pad5)
- Y1 pad 2: Net-(C3-Pad1) -> GND
Routing:
- net /MACRO2: track 53.3 -> 0.00 mm
- net /MACRO_1: track 52.5 -> 0.00 mm
- net GND: track 85.9 -> 76.6 mm, vias 61 -> 52
- net Net-(C3-Pad1): track 9.49 -> 5.24 mm
- net /XIN: track 14.5 -> 11.9 mm
Other:
- rule pad_to_mask_clearance: 0.051 -> 0
