File: hw/minigeki.kicad_sch (KiCad schematic)
At the start: 61 parts, among them J1 USB_C_Receptacle_USB2.0, J2 Conn_01x02, SW1 LEFT_G, SW10 RIGHT_G, SW11 RIGHT_START, SW12 MACRO_1, SW2 LEFT_START, SW3 RIGHT_R, SW4 RIGHT_B, SW5 RIGHT_WALL, SW6 MACRO_2, SW7 LEFT_R, SW8 LEFT_B, SW9 LEFT_WALL, U1 NCP1117-3.3_SOT223, U2 W25Q128JVS, U3 RP2040, Y1 ABLS-12.000MHZ-B4-T

Commit message: hw: finish main routing
Parts:
- added C26: 100n, Capacitor_SMD:C_0402_1005Metric, symbol Device:C
- renumbered SW7 to SW1, SW5 to SW10, SW12 to SW11, SW6 to SW12, SW1 to SW2, SW8 to SW3, SW2 to SW4, SW9 to SW5, SW3 to SW6, SW10 to SW7, SW4 to SW8, SW11 to SW9
Connections:
- net GPIO24 is gone; now on net LED_DIN: U3.36 (GPIO24)
- net GND: now also C26.1; no longer SW5.2
- net VBUS: now also C26.2
- net GPIO0: no longer names the net of U3.2 (GPIO0)
- net GPIO0: no longer SW1.1
- net GPIO1: no longer names the net of U3.3 (GPIO1)
- net GPIO1: no longer SW2.1
- net GPIO10: no longer names the net of U3.13 (GPIO10)
- net GPIO10: no longer SW11.1
- net GPIO11: no longer names the net of U3.14 (GPIO11)
- net GPIO11: no longer SW12.1
- net GPIO12 renamed RIGHT_B
- net RIGHT_B: now also SW8.1
- net GPIO13 renamed RIGHT_G
- net RIGHT_G: now also SW7.1
- net GPIO14 renamed RIGHT_R
- net RIGHT_R: now also SW6.1
- net GPIO15: no longer names the net of U3.18 (GPIO15)
- net GPIO16: no longer names the net of U3.27 (GPIO16)
- net GPIO17: no longer names the net of U3.28 (GPIO17)
- net GPIO18 renamed LEFT_B
- net LEFT_B: now also SW3.1
- net GPIO19 renamed LEFT_G
- net LEFT_G: now also SW2.1
- net GPIO2: no longer names the net of U3.4 (GPIO2)
- net GPIO2: no longer SW3.1
- net GPIO20 renamed LEFT_R
- net LEFT_R: now also SW1.1
- net GPIO21: no longer names the net of U3.32 (GPIO21)
- net GPIO22: no longer names the net of U3.34 (GPIO22)
- net GPIO23: no longer names the net of U3.35 (GPIO23)
- net GPIO25: no longer names the net of U3.37 (GPIO25)
- net GPIO27_ADC1 renamed MACRO_1
- net MACRO_1: now also SW11.1
- net GPIO28_ADC2 renamed LEFT_WALL
- net LEFT_WALL: now also SW5.1
- net GPIO29_ADC3 renamed LEFT_START
- net LEFT_START: now also SW4.1
- net GPIO3: no longer names the net of U3.5 (GPIO3)
- net GPIO3: no longer SW4.1
- net GPIO4 renamed RIGHT_START
- net RIGHT_START: now also SW9.1; no longer SW5.1
- net GPIO5 renamed RIGHT_WALL
- net RIGHT_WALL: now also SW10.1; no longer SW6.1
- net GPIO6 renamed MACRO2
- net MACRO2: now also SW12.1; no longer SW7.1
- net GPIO7: no longer names the net of U3.9 (GPIO7)
- net GPIO7: no longer SW8.1
- net GPIO8: no longer names the net of U3.11 (GPIO8)
- net GPIO8: no longer SW9.1
- net GPIO9: no longer names the net of U3.12 (GPIO9)
- net GPIO9: no longer SW10.1
- no-connect marks 20 -> 19
Other:
- moved on the sheet: SW1, SW10, SW11, SW12, SW2, SW3, SW4, SW5, SW6, SW7, SW8, SW9

Commit message: hw: update schematic to reflect PCB changes
Connections:
- net GND: now also SW5.2
Changed lines of the file:
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@@
   (junction (at 74.93 30.48) (diameter 0) (color 0 0 0 0)
+  )
+  (junction (at 367.03 133.35) (diameter 0) (color 0 0 0 0)
   )
   (junction (at 271.78 209.55) (diameter 0) (color 0 0 0 0)
@@
     (stroke (width 0) (type default) (color 0 0 0 0))
   )
+  (wire (pts (xy 367.03 133.35) (xy 367.03 138.43))
+    (stroke (width 0) (type default) (color 0 0 0 0))
+  )
   (wire (pts (xy 44.45 125.73) (xy 31.75 125.73))
     (stroke (width 0) (type default) (color 0 0 0 0))
@@
     (stroke (width 0) (type default) (color 0 0 0 0))
   )
+  (wire (pts (xy 359.41 133.35) (xy 367.03 133.35))
+    (stroke (width 0) (type default) (color 0 0 0 0))
+  )
   (wire (pts (xy 45.72 38.1) (xy 49.53 38.1))
     (stroke (width 0) (type default) (color 0 0 0 0))
@@
     (stroke (width 0) (type default) (color 0 0 0 0))
   )
-  (wire (pts (xy 367.03 128.27) (xy 367.03 138.43))
-    (stroke (width 0) (type default) (color 0 0 0 0))
-  )
+  (wire (pts (xy 367.03 128.27) (xy 367.03 133.35))
+    (stroke (width 0) (type default) (color 0 0 0 0))
+  )

Commit message: hw: add mounting holes, flip components to top of the board
Parts:
- added H1, H2, H3, H4, H5, H6: MountingHole_Pad, MountingHole:MountingHole_2.2mm_M2_Pad_TopOnly, symbol Mechanical:MountingHole_Pad
Connections:
- net GND: now also H1.1, H2.1, H3.1, H4.1, H5.1, H6.1
Other:
- note added: "Mounting holes for top board/plate"
- company: Raspberry Pi (Trading) Ltd -> defvs
- title: RP2040 Minimal Design Example -> m.i.n.i.g.e.k.i

Commit message: hw: final PCB for v3.0
Parts:
- H1, H2, H3, H4, H5, H6: now left out of the parts list
Connections:
- net LED_DIN: now also U3.3 (GPIO1); no longer U3.36 (GPIO24)
- net LEFT_B: now also U3.8 (GPIO6); no longer U3.29 (GPIO18)
- net LEFT_G: now also U3.7 (GPIO5); no longer U3.30 (GPIO19)
- net LEFT_R: now also U3.6 (GPIO4); no longer U3.31 (GPIO20)
- net LEFT_START: now also U3.2 (GPIO0); no longer U3.41 (GPIO29_ADC3)
- net LEFT_WALL: now also U3.4 (GPIO2); no longer U3.40 (GPIO28_ADC2)
- net MACRO2: now also U3.32 (GPIO21); no longer U3.8 (GPIO6)
- net MACRO_1: now also U3.5 (GPIO3); no longer U3.39 (GPIO27_ADC1)
- net RIGHT_B: now also U3.31 (GPIO20); no longer U3.15 (GPIO12)
- net RIGHT_G: now also U3.30 (GPIO19); no longer U3.16 (GPIO13)
- net RIGHT_R: now also U3.29 (GPIO18); no longer U3.17 (GPIO14)
- net RIGHT_START: now also U3.35 (GPIO23); no longer U3.6 (GPIO4)
- net RIGHT_WALL: now also U3.34 (GPIO22); no longer U3.7 (GPIO5)

Commit message: hw: final prototype export
Parts:
- removed SW11: MACRO_1, Button_Switch_SMD:SW_SPST_PTS810, symbol Switch:SW_Push
- removed SW12: MACRO_2, Button_Switch_SMD:SW_SPST_PTS810, symbol Switch:SW_Push
- removed Y1: ABLS-12.000MHZ-B4-T, RP2040_minimal:Crystal_SMD_HC49-US, symbol Device:Crystal
- added Y1: Q22FA23V0041800, Crystal:Crystal_SMD_3225-4Pin_3.2x2.5mm, symbol Device:Crystal_GND24
- C1, C4: Package (none) -> 0805
- C10, C11, C12, C13, C14, C15, C16, C17, C18, C19, C2, C20, C21, C22, C23, C24, C25, C26, C3, C5, C6, C7, C8, C9, R1, R2, R3, R4, R5, R6, R7: Package (none) -> 0402
- D1, D10, D2, D3, D4, D5, D6, D7, D8, D9: MPN (none) -> SK6812MINI; Package (none) -> PLCC4_3.5x3.5mm_P1.75mm
- J1: MPN (none) -> U262-161N-4BVC11; Package (none) -> U262-161N-4BVC11
- RV1: MPN (none) -> PTA4543-2015DPB103
- U1: MPN (none) -> NCP1117ST33T3G; Package (none) -> SOT223-3
- U2: MPN (none) -> W25Q128JVS; Package (none) -> SOIC-8_5.23x5.23mm_P1.27mm
- U3: MPN (none) -> RP2040; Package (none) -> QFN-56
Connections:
- net GND: now also Y1.2, Y1.4
- net XIN: now also Y1.1
- net at C3.1, R5.2: now also Y1.3
- net MACRO2: no longer names the net of U3.32 (GPIO21)
- net MACRO_1: no longer names the net of U3.5 (GPIO3)
- no-connect marks 19 -> 21
